Commit message: ROS TASK #1

File: src/firstbot/urdf/simple_bot.xacro (robot description, xacro)
@@ -24,4 +24,7 @@
     </inertial>
   </link>
+  <gazebo reference="base_link">
+      <material>Gazebo/White</material>
+  </gazebo>
 <link name="right_front_wheel">
   <!--origin xyz="0.1 -0.13 0.1" rpy="0 1.5707 1.5707"/-->
@@ -49,4 +52,7 @@
     </inertial>
   </link>
+  <gazebo reference="right_front_wheel">
+      <material>Gazebo/Black</material>
+  </gazebo>
 <joint name="right_front_wheel_joint" type="continuous">
     <parent link="body"/>
@@ -55,5 +61,5 @@
     <axis xyz="0 1 0" rpy="0 0 0"/>
     <limit effort="100" velocity="100"/>
-    <joint_properties damping="0.0" friction="0.0"/>
+    <joint_properties damping="1.0" friction="1.0"/>
   </joint>
 <link name="left_front_wheel">
@@ -82,4 +88,7 @@
     </inertial>
   </link>
+  <gazebo reference="left_front_wheel">
+      <material>Gazebo/Black</material>
+  </gazebo>
 <joint name="left_front_wheel_joint" type="continuous">
     <parent link="body"/>
@@ -88,5 +97,5 @@
     <axis xyz="0 1 0" rpy="0 0 0"/>
     <limit effort="100" velocity="100"/>
-    <joint_properties damping="0.0" friction="0.0"/>
+    <joint_properties damping="1.0" friction="1.0"/>
   </joint>
 <link name="right_rear_wheel">
@@ -115,4 +124,7 @@
     </inertial>
   </link>
+  <gazebo reference="right_rear_wheel">
+      <material>Gazebo/Black</material>
+  </gazebo>
 <joint name="right_rear_wheel_joint" type="continuous">
     <parent link="body"/>
@@ -121,5 +133,5 @@
     <axis xyz="0 1 0" rpy="0 0 0"/>
     <limit effort="100" velocity="100"/>
-    <joint_properties damping="0.0" friction="0.0"/>
+    <joint_properties damping="1.0" friction="1.0"/>
   </joint>
 <link name="left_rear_wheel">
@@ -148,4 +160,7 @@
     </inertial>
   </link>
+  <gazebo reference="left_rear_wheel">
+      <material>Gazebo/Black</material>
+  </gazebo>
 <joint name="left_rear_wheel_joint" type="continuous">
     <parent link="body"/>
@@ -154,5 +169,25 @@
     <axis xyz="0 1 0" rpy="0 0 0"/>
     <limit effort="100" velocity="100"/>
-    <joint_properties damping="0.0" friction="0.0"/>
+    <joint_properties damping="1.0" friction="1.0"/>
   </joint>
+  <gazebo>
+    <plugin name="differential_drive_controller" filename="libgazebo_ros_diff_drive.so">
+      <legacyMode>false</legacyMode>
+      <alwaysOn>true</alwaysOn>
+      <updateRate>20</updateRate>
+      <leftFrontJoint>left_front_wheel_joint</leftFrontJoint>
+      <rightFrontJoint>right_front_wheel_joint</rightFrontJoint>
+      <leftRearJoint>left_rear_wheel_joint</leftRearJoint>
+      <rightRearJoint>right_rear_wheel_joint</rightRearJoint>
+      <wheelSeparation>0.4</wheelSeparation>
+      <wheelDiameter>0.1</wheelDiameter>
+      <torque>20</torque>
+      <commandTopic>cmd_vel</commandTopic>
+      <odometryTopic>odom</odometryTopic>
+      <odometryFrame>odom</odometryFrame>
+      <robotBaseFrame>body</robotBaseFrame>
+    </plugin>
+  </gazebo>
+  <gazebo reference="body">
+    </gazebo>
 </robot>
